Commit message: Updated robot description params

File: rox_description/urdf/xacros/argo_caster.xacro (robot description, xacro)
@@ -11,5 +11,5 @@
     <inertial>
     <!-- These are not accurate value -->
-      <mass value="0.025" />
+      <mass value="3.025" />
       <origin xyz="${vis_pos}" rpy="${vis_rot}" />
       <inertia ixx="0.02" ixy="0" ixz="0" iyy="0.0" iyz="0" izz="0.02" />

File: rox_description/urdf/xacros/argo_wheel.xacro (robot description, xacro)
@@ -11,5 +11,5 @@
     <inertial>
     <!-- These are not accurate value -->
-      <mass value="5" />
+      <mass value="10" />
       <origin xyz="0 0 0" rpy="0 0 0"/>
       <inertia ixx="0.02" ixy="0" ixz="0" iyy="0.02" iyz="0" izz="0.02" />

File: rox_description/urdf/xacros/frame.xacro (robot description, xacro)
@@ -13,7 +13,5 @@
         <mass value="140.0" />
         <origin xyz="0.0 0 0.18" rpy="0.0 0.0 0.0"/>
-        <inertia ixx="0.299" ixy="0.0" ixz="0.0"
-                 iyy="0.351" iyz="0.0"
-                 izz="0.360" />
+        <inertia ixx="7.8" ixy="0.0" ixz="0" iyy="7.8" iyz="0.0" izz="7.8"/>
       </inertial>
       <visual>
