Commit message: Updated frame mass to fix the tipping over issue when navigating

File: rox_description/urdf/xacros/frame.xacro (robot description, xacro)
@@ -11,5 +11,5 @@
       <inertial>
       <!-- These are not accurate value -->
-        <mass value="8.0" />
+        <mass value="140.0" />
         <origin xyz="0.0 0 0.18" rpy="0.0 0.0 0.0"/>
         <inertia ixx="0.299" ixy="0.0" ixz="0.0"

Commit message: UR ams ros2_control support for rox platform (#36)
* Added ros2_control nodes to launch file for arm simulation, modified urdf to support ros2_control, added config files

* added missing commits

* fixed typo in launch file

* Updated frame mass to fix the tipping over issue when navigating

* Updated robot description params

File: rox_description/urdf/xacros/frame.xacro (robot description, xacro)
@@ -11,9 +11,7 @@
       <inertial>
       <!-- These are not accurate value -->
-        <mass value="8.0" />
+        <mass value="140.0" />
         <origin xyz="0.0 0 0.18" rpy="0.0 0.0 0.0"/>
-        <inertia ixx="0.299" ixy="0.0" ixz="0.0"
-                 iyy="0.351" iyz="0.0"
-                 izz="0.360" />
+        <inertia ixx="7.8" ixy="0.0" ixz="0" iyy="7.8" iyz="0.0" izz="7.8"/>
       </inertial>
       <visual>

Commit message: updated use_sim_time argument in launch file and frame origin

File: rox_description/urdf/xacros/frame.xacro (robot description, xacro)
@@ -12,5 +12,5 @@
       <!-- These are not accurate value -->
         <mass value="140.0" />
-        <origin xyz="0.0 0 0.18" rpy="0.0 0.0 0.0"/>
+        <origin xyz="0.0 0.0 0.0" rpy="0.0 0.0 0.0"/>
         <inertia ixx="7.8" ixy="0.0" ixz="0" iyy="7.8" iyz="0.0" izz="7.8"/>
       </inertial>
