Commit message: updating EMROX for caroline

File: rox_description/urdf/rox.urdf.xacro (robot description, xacro)
@@ -10,4 +10,5 @@
     <xacro:arg name="use_imu" default="false"/>
     <xacro:arg name="use_d435" default="false"/>
+    <xacro:arg name="use_ur_dc" default="false"/>
     <!-- Xacro Properties -->
     <xacro:property name="frame" value="$(arg frame_type)"/>
@@ -20,4 +21,5 @@
     <xacro:property name="imu" value="$(arg use_imu)"/>
     <xacro:property name="d435" value="$(arg use_d435)"/>
+    <xacro:property name="ur_dc" value="$(arg use_ur_dc)"/>
     <!-- Include xacro files -->
     <xacro:include filename="$(find rox_description)/urdf/xacros/frame.xacro" />
@@ -105,4 +107,10 @@
     <!-- arm -->
     <xacro:unless value="${arm == ''}">
+        <xacro:if value="${ur_dc == False}">
+            <xacro:property name="arm_height" value="0.46" />
+        </xacro:if>
+        <xacro:if value="${ur_dc == True}">
+            <xacro:property name="arm_height" value="0.276" />
+        </xacro:if>
         <xacro:include filename="$(find rox_description)/urdf/xacros/cabinet.xacro" />
         <xacro:cabinet name="cabinet" parent="base_footprint">
@@ -143,5 +151,5 @@
                 >
                 <!-- position robot in the world -->
-                <origin xyz="0.133 0.0 0.416" rpy="0.0 0.0 -1.5708" />
+                <origin xyz="0.218 0.0 ${arm_height}" rpy="0.0 0.0 -1.5708" />
             </xacro:ur_robot>
         </xacro:if>

Commit message: updating EMROX for caroline

File: rox_description/urdf/rox.urdf.xacro (robot description, xacro)
@@ -10,4 +10,5 @@
     <xacro:arg name="use_imu" default="false"/>
     <xacro:arg name="use_d435" default="false"/>
+    <xacro:arg name="use_ur_dc" default="false"/>
     <!-- Xacro Properties -->
     <xacro:property name="frame" value="$(arg frame_type)"/>
@@ -20,4 +21,5 @@
     <xacro:property name="imu" value="$(arg use_imu)"/>
     <xacro:property name="d435" value="$(arg use_d435)"/>
+    <xacro:property name="ur_dc" value="$(arg use_ur_dc)"/>
     <!-- Include xacro files -->
     <xacro:include filename="$(find rox_description)/urdf/xacros/frame.xacro" />
@@ -105,4 +107,10 @@
     <!-- arm -->
     <xacro:unless value="${arm == ''}">
+        <xacro:if value="${ur_dc == False}">
+            <xacro:property name="arm_height" value="0.46" />
+        </xacro:if>
+        <xacro:if value="${ur_dc == True}">
+            <xacro:property name="arm_height" value="0.276" />
+        </xacro:if>
         <xacro:include filename="$(find rox_description)/urdf/xacros/cabinet.xacro" />
         <xacro:cabinet name="cabinet" parent="base_footprint">
@@ -133,5 +141,5 @@
                 >
                 <!-- position robot in the world -->
-                <origin xyz="0.133 0.0 0.416" rpy="0.0 0.0 -1.5708" />
+                <origin xyz="0.218 0.0 ${arm_height}" rpy="0.0 0.0 -1.5708" />
             </xacro:ur_robot>
         </xacro:if>

File: rox_description/urdf/xacros/cabinet.xacro (robot description, xacro)
@@ -2,10 +2,16 @@
 <robot xmlns:xacro="http://www.ros.org/wiki/xacro" name="rox">
   <xacro:macro name="cabinet" params="name parent *origin">
-   <joint name="${name}_joint" type="fixed">
+    <joint name="${name}_joint" type="fixed">
     <xacro:insert_block name="origin" />
     <joint_properties damping="1" friction="1" />
     <parent link="${parent}" />
     <child link="${name}_link" />
-   </joint>
+    </joint>
+    <xacro:if value="${ur_dc == True}">
+      <xacro:property name="cabinet_mesh" value="cabinet_dc" />
+    </xacro:if>
+    <xacro:if value="${ur_dc == False}">
+      <xacro:property name="cabinet_mesh" value="cabinet_ac" />
+    </xacro:if>
     <link name="${name}_link">
       <inertial>
@@ -19,5 +25,5 @@
         <origin xyz="0 0 0" rpy="0 0 0" />
         <geometry>
-            <mesh filename="package://rox_description/meshes/cabinet.dae" scale="0.1 0.1 0.1"/>
+          <mesh filename="package://rox_description/meshes/${cabinet_mesh}.dae" scale="0.1 0.1 0.1"/>
         </geometry>
       </visual>
@@ -25,5 +31,5 @@
         <origin xyz="0. 0. 0" rpy="0 0 0" />
         <geometry>
-            <mesh filename="package://rox_description/meshes/cabinet.dae" scale="0.1 0.1 0.1"/>
+          <mesh filename="package://rox_description/meshes/${cabinet_mesh}.dae" scale="0.1 0.1 0.1"/>
         </geometry>
       </collision>

Commit message: updating the orientation for ur arm

File: rox_description/urdf/rox.urdf.xacro (robot description, xacro)
@@ -151,5 +151,5 @@
                 >
                 <!-- position robot in the world -->
-                <origin xyz="0.218 0.0 ${arm_height}" rpy="0.0 0.0 -1.5708" />
+                <origin xyz="0.218 0.0 ${arm_height}" rpy="0.0 0.0 3.1415926535897931" />
             </xacro:ur_robot>
         </xacro:if>

Commit message: updating the orientation for ur arm

File: rox_description/urdf/rox.urdf.xacro (robot description, xacro)
@@ -141,5 +141,5 @@
                 >
                 <!-- position robot in the world -->
-                <origin xyz="0.218 0.0 ${arm_height}" rpy="0.0 0.0 -1.5708" />
+                <origin xyz="0.218 0.0 ${arm_height}" rpy="0.0 0.0 3.1415926535897931" />
             </xacro:ur_robot>
         </xacro:if>

Commit message: updating xacro

File: rox_description/urdf/rox.urdf.xacro (robot description, xacro)
@@ -119,4 +119,6 @@
         <xacro:if value="${use_ur_arm == True}">
             <xacro:include filename="$(find ur_description)/urdf/ur_macro.xacro"/>
+            <xacro:include filename="$(find ur_robot_driver)/urdf/ur.ros2_control.xacro" />
+            <xacro:include filename="$(find ur_description)/urdf/inc/ur_transmissions.xacro" />
             <xacro:arg name="tf_prefix" default="${arm}" />
             <xacro:arg name="joint_limit_params" default="$(find ur_description)/config/$(arg arm_type)/joint_limits.yaml"/>
@@ -124,9 +126,32 @@
             <xacro:arg name="physical_params" default="$(find ur_description)/config/$(arg arm_type)/physical_parameters.yaml"/>
             <xacro:arg name="visual_params" default="$(find ur_description)/config/$(arg arm_type)/visual_parameters.yaml"/>
-            <xacro:arg name="transmission_hw_interface" default=""/>
-            <xacro:arg name="safety_limits" default="false"/>
+            <xacro:arg name="initial_positions_file" default="$(find ur_description)/config/initial_positions.yaml"/>
+            <xacro:arg name="transmission_hw_interface" default="hardware_interface/PositionJointInterface"/>
+            <xacro:arg name="safety_limits" default="true"/>
             <xacro:arg name="safety_pos_margin" default="0.15"/>
             <xacro:arg name="safety_k_position" default="20"/>
             <xacro:arg name="force_abs_paths" default="false" />
+            <!-- ros2_control related parameters -->
+            <xacro:arg name="headless_mode" default="false" />
+            <xacro:arg name="robot_ip" default="192.168.1.102" />
+            <xacro:arg name="script_filename" default="$(find ur_client_library)/resources/external_control.urscript"/>
+            <xacro:arg name="output_recipe_filename" default="$(find ur_robot_driver)/resources/rtde_output_recipe.txt"/>
+            <xacro:arg name="input_recipe_filename" default="$(find ur_robot_driver)/resources/rtde_input_recipe.txt"/>
+            <xacro:arg name="reverse_ip" default="0.0.0.0"/>
+            <xacro:arg name="script_command_port" default="50004"/>
+            <xacro:arg name="reverse_port" default="50001"/>
+            <xacro:arg name="script_sender_port" default="50002"/>
+            <xacro:arg name="trajectory_port" default="50003"/>
+            <!--   tool communication related parameters-->
+            <xacro:arg name="use_tool_communication" default="false" />
+            <xacro:arg name="tool_voltage" default="0" />
+            <xacro:arg name="tool_parity" default="0" />
+            <xacro:arg name="tool_baud_rate" default="115200" />
+            <xacro:arg name="tool_stop_bits" default="1" />
+            <xacro:arg name="tool_rx_idle_chars" default="1.5" />
+            <xacro:arg name="tool_tx_idle_chars" default="3.5" />
+            <xacro:arg name="tool_device_name" default="/tmp/ttyUR" />
+            <xacro:arg name="tool_tcp_port" default="54321" />
+            <xacro:property name="initial_positions_file" default="$(arg initial_positions_file)"/>
             <xacro:ur_robot name="${arm}"
                 parent="cabinet_link"
@@ -143,4 +168,30 @@
                 <origin xyz="0.218 0.0 ${arm_height}" rpy="0.0 0.0 3.1415926535897931" />
             </xacro:ur_robot>
+            <xacro:ur_ros2_control
+                name="ur10e"
+                tf_prefix="$(arg tf_prefix)"
+                kinematics_parameters_file="$(arg kinematics_params)"
+                transmission_hw_interface="$(arg transmission_hw_interface)"
+                headless_mode="$(arg headless_mode)"
+                initial_positions="${xacro.load_yaml(initial_positions_file)}"
+                use_tool_communication="$(arg use_tool_communication)"
+                tool_voltage="$(arg tool_voltage)"
+                tool_parity="$(arg tool_parity)"
+                tool_baud_rate="$(arg tool_baud_rate)"
+                tool_stop_bits="$(arg tool_stop_bits)"
+                tool_rx_idle_chars="$(arg tool_rx_idle_chars)"
+                tool_tx_idle_chars="$(arg tool_tx_idle_chars)"
+                tool_device_name="$(arg tool_device_name)"
+                tool_tcp_port="$(arg tool_tcp_port)"
+                robot_ip="$(arg robot_ip)"
+                script_filename="$(arg script_filename)"
+                output_recipe_filename="$(arg output_recipe_filename)"
+                input_recipe_filename="$(arg input_recipe_filename)"
+                reverse_ip="$(arg reverse_ip)"
+                script_command_port="$(arg script_command_port)"
+                reverse_port="$(arg reverse_port)"
+                script_sender_port="$(arg script_sender_port)"
+                trajectory_port="$(arg trajectory_port)"
+            />
         </xacro:if>
     </xacro:unless>

Commit message: added missing commits

File: rox_description/urdf/rox.urdf.xacro (robot description, xacro)
@@ -121,4 +121,12 @@
             <xacro:arg name="safety_k_position" default="20"/>
             <xacro:arg name="force_abs_paths" default="false" />
+            <xacro:arg name="sim_ignition" default="$(arg use_gz)" />
+            <xacro:arg name="simulation_controllers" default="$(find rox_bringup)/configs/ur_config/$(arg arm_type)/ur_controllers.yaml"/>
+            <xacro:arg name="initial_positions_file" default="$(find rox_bringup)/configs/ur_config/initial_joint_positions.yaml"/>
+           <!-- parse initial positions as a dictionary -->
+            <xacro:property
+                name="ur_initial_positions"
+                value="${xacro.load_yaml('$(arg initial_positions_file)')}"
+                />
             <xacro:ur_robot name="${arm}"
                 parent="cabinet_link"
@@ -131,4 +139,6 @@
                 safety_pos_margin="$(arg safety_pos_margin)"
                 safety_k_position="$(arg safety_k_position)"
+                sim_ignition="$(arg sim_ignition)"
+                initial_positions = "${ur_initial_positions}"
                 >
                 <!-- position robot in the world -->
@@ -141,4 +151,14 @@
         <xacro:include filename="$(find rox_description)/urdf/xacros/gazebo.xacro" />
         <xacro:gazebo_plugins />
+        <xacro:if value="${use_ur_arm == True}">
+            <gazebo reference="cabinet_link">
+            </gazebo>
+            <gazebo>
+                <plugin filename="libgz_ros2_control-system.so" name="gz_ros2_control::GazeboSimROS2ControlPlugin">
+                    <parameters>$(arg simulation_controllers)</parameters>
+                    <controller_manager_node_name>$(arg tf_prefix)controller_manager</controller_manager_node_name>
+                </plugin>
+            </gazebo>
+        </xacro:if>
     </xacro:if>
 </robot>

Commit message: Cherry picked changes for adding ac and dc variant option and modified arm position to fit ac cabinet version

File: rox_description/urdf/rox.urdf.xacro (robot description, xacro)
@@ -108,5 +108,6 @@
     <xacro:unless value="${arm == ''}">
         <xacro:if value="${ur_dc == False}">
-            <xacro:property name="arm_height" value="0.46" />
+            <!-- Different height for AC arm-->
+            <xacro:property name="arm_height" value="0.376" />
         </xacro:if>
         <xacro:if value="${ur_dc == True}">

Commit message: Ac and Dc variant UR arm support for ROX  (#40)
* Added ros2_control nodes to launch file for arm simulation, modified urdf to support ros2_control, added config files

* added missing commits

* fixed typo in launch file

* Updated frame mass to fix the tipping over issue when navigating

* Updated robot description params

* updated use_sim_time argument in launch file and frame origin

* updating EMROX for caroline

* updating argo to caroline

* updating bringup with the DC variant option selection for UR

* updating the orientation for ur arm

* Cherry picked changes for adding ac and dc variant option and modified arm position to fit ac cabinet version

* Updated README with launch commands

* Removed unnecessary files, updated README and launch file

* Delete rox_bringup/configs/ur_config/ur10/moveit_controllers.yaml

* Delete rox_bringup/configs/ur_config/ompl_planning.yaml

---------

Co-authored-by: Pradheep <padhupradheep@gmail.com>

File: rox_description/urdf/rox.urdf.xacro (robot description, xacro)
@@ -10,4 +10,5 @@
     <xacro:arg name="use_imu" default="false"/>
     <xacro:arg name="use_d435" default="false"/>
+    <xacro:arg name="use_ur_dc" default="false"/>
     <!-- Xacro Properties -->
     <xacro:property name="frame" value="$(arg frame_type)"/>
@@ -20,4 +21,5 @@
     <xacro:property name="imu" value="$(arg use_imu)"/>
     <xacro:property name="d435" value="$(arg use_d435)"/>
+    <xacro:property name="ur_dc" value="$(arg use_ur_dc)"/>
     <!-- Include xacro files -->
     <xacro:include filename="$(find rox_description)/urdf/xacros/frame.xacro" />
@@ -105,4 +107,11 @@
     <!-- arm -->
     <xacro:unless value="${arm == ''}">
+        <xacro:if value="${ur_dc == False}">
+            <!-- Different height for AC arm-->
+            <xacro:property name="arm_height" value="0.376" />
+        </xacro:if>
+        <xacro:if value="${ur_dc == True}">
+            <xacro:property name="arm_height" value="0.276" />
+        </xacro:if>
         <xacro:include filename="$(find rox_description)/urdf/xacros/cabinet.xacro" />
         <xacro:cabinet name="cabinet" parent="base_footprint">
@@ -122,5 +131,5 @@
             <xacro:arg name="force_abs_paths" default="false" />
             <xacro:arg name="sim_ignition" default="$(arg use_gz)" />
-            <xacro:arg name="simulation_controllers" default="$(find rox_bringup)/configs/ur_config/$(arg arm_type)/ur_controllers.yaml"/>
+            <xacro:arg name="simulation_controllers" default=""/>
             <xacro:arg name="initial_positions_file" default="$(find rox_bringup)/configs/ur_config/initial_joint_positions.yaml"/>
            <!-- parse initial positions as a dictionary -->
@@ -143,5 +152,5 @@
                 >
                 <!-- position robot in the world -->
-                <origin xyz="0.133 0.0 0.416" rpy="0.0 0.0 -1.5708" />
+                <origin xyz="0.218 0.0 ${arm_height}" rpy="0.0 0.0 3.1415926535897931" />
             </xacro:ur_robot>
         </xacro:if>

Commit message: Removed meca configuration and frame_type arg from bringup_sim_launch.py, bringup_launch.py, and description_launch.py. Removed type param from frame.xacro. Removed frame_type arg and frame and frame_len property from rox.urdf.xacro. Renamed short_frame.dae to frame.dae and removed long_frame.dae. Removed frame_len property from argo_drive.xacro, diff_drive.xacro, and trike_drive.xacro.

File: rox_description/urdf/rox.urdf.xacro (robot description, xacro)
@@ -2,5 +2,4 @@
 <robot xmlns:xacro="http://www.ros.org/wiki/xacro" name="rox">
     <!-- Xacro Arguments-->
-    <xacro:arg name="frame_type" default="short"/>
     <xacro:arg name="rox_type" default="argo"/>
     <xacro:arg name="joint_type" default="fixed"/>
@@ -14,5 +13,4 @@
     <xacro:arg name="force_abs_paths" default="false"/>
     <!-- Xacro Properties -->
-    <xacro:property name="frame" value="$(arg frame_type)"/>
     <xacro:property name="rox_typ" default="$(arg rox_type)"/>
     <xacro:property name="joint_typ" value="$(arg joint_type)"/>
@@ -34,15 +32,7 @@
         <xacro:property name="use_arm" value="true"/>
     </xacro:if>
-    <!-- Assigning Xacro properties -->
-    <xacro:if value="${frame == 'short'}">
-        <xacro:property name="frame_len" value="0.0" />
-    </xacro:if>
-    <xacro:if value="${frame == 'long'}">
-        <xacro:property name="frame_len" value="0.13" />
-    </xacro:if>
     <!-- Building the robot from here -->
     <link name="base_link" />
-    <xacro:rox_base name="base_footprint"  parent="base_link"
-        type="${frame}">
+    <xacro:rox_base name="base_footprint"  parent="base_link">
         <origin xyz="0 0 0" rpy="0 0 0" />
     </xacro:rox_base>
@@ -70,8 +60,8 @@
     <xacro:if value="${scanner_typ == 'nanoscan'}">
         <xacro:sick_nanoscan name="lidar_1" parent="base_link">
-            <origin rpy="${pi} 0 ${pi/4}" xyz="${0.2995 + frame_len} 0.269 0.189"/>
+            <origin rpy="${pi} 0 ${pi/4}" xyz="${0.2995} 0.269 0.189"/>
         </xacro:sick_nanoscan>
         <xacro:sick_nanoscan name="lidar_2" parent="base_link">
-            <origin rpy="${pi} 0 -${pi - pi/4}" xyz="-${0.2995 - frame_len} -0.269 0.189"/>
+            <origin rpy="${pi} 0 -${pi - pi/4}" xyz="-${0.2995} -0.269 0.189"/>
         </xacro:sick_nanoscan>
     </xacro:if>
@@ -79,8 +69,8 @@
     <xacro:if value="${scanner_typ == 'psenscan'}">
         <xacro:pilz_psenscan name="lidar_1" parent="base_link">
-            <origin rpy="0 0 ${pi/4}" xyz="${0.3016 + frame_len} 0.2719 0.191"/>
+            <origin rpy="0 0 ${pi/4}" xyz="${0.3016} 0.2719 0.191"/>
         </xacro:pilz_psenscan>
         <xacro:pilz_psenscan name="lidar_2" parent="base_link">
-            <origin rpy="0 0 -${pi - pi/4}" xyz="-${0.3016 + frame_len} -0.2719 0.191"/>
+            <origin rpy="0 0 -${pi - pi/4}" xyz="-${0.3016} -0.2719 0.191"/>
         </xacro:pilz_psenscan>
     </xacro:if>
@@ -113,5 +103,5 @@
         <xacro:include filename="$(find rox_description)/urdf/xacros/cabinet.xacro" />
         <xacro:cabinet name="cabinet" parent="base_footprint">
-            <origin rpy="0 0 0" xyz="${frame_len} 0 0.33"/>
+            <origin rpy="0 0 0" xyz="0 0 0.33"/>
         </xacro:cabinet>
         <!-- Universal Robotics (UR) Arms-->

File: rox_description/urdf/xacros/frame.xacro (robot description, xacro)
@@ -1,5 +1,5 @@
 <?xml version="1.0"?>
 <robot xmlns:xacro="http://www.ros.org/wiki/xacro" name="rox">
-  <xacro:macro name="rox_base" params="name parent type *origin">
+  <xacro:macro name="rox_base" params="name parent *origin">
    <joint name="${name}_joint" type="fixed">
     <xacro:insert_block name="origin" />
@@ -18,5 +18,5 @@
         <origin xyz="0.0 0.0 0.0" rpy="0 0 0" />
         <geometry>
-          <mesh filename="package://rox_description/meshes/${type}_frame.dae" scale="0.1 0.1 0.1"/>
+          <mesh filename="package://rox_description/meshes/frame.dae" scale="0.1 0.1 0.1"/>
         </geometry>
       </visual>
@@ -24,5 +24,5 @@
         <origin xyz="0.0 0.0 0.0" rpy="0 0 0"/>
         <geometry>
-          <mesh filename="package://rox_description/meshes/${type}_frame.dae" scale="0.1 0.1 0.1"/>
+          <mesh filename="package://rox_description/meshes/frame.dae" scale="0.1 0.1 0.1"/>
         </geometry>
       </collision>
